Commit message: [fixed]Collision

File: z1/urdf/z1.urdf (robot description, URDF)
Before this commit: robot z1_description, 10 links, 9 joints
Links:
- link gripperMover: geometry collision mesh filename=../meshes/visual/z1_GripperMover.stl scale=1 1 1; visual mesh filename=../meshes/visual/z1_GripperMover.stl scale=1 1 1
- link gripperStator: geometry collision cylinder length=0.051 radius=0.0325; collision mesh filename=../meshes/visual/z1_GripperStator.stl scale=1 1 1
